Commit message: [feature] merge 2 sim and final structure

File: UAV_models/moving_target/moving_target.urdf (robot description, URDF)
Before this commit: robot moving_target, 5 links, 4 joints
Links:
- added link raruco_marker_link, mass 0.05; collision box size=0.4 0.4 0.002; visual mesh filename=package://uav_models/moving_target/marker_plate.obj scale=0.4 0.4 1.0
Joints:
- added joint raruco_marker_joint: type fixed, parent base_link, child raruco_marker_link, origin xyz=0 0 0.221 rpy=0 0 0
