Commit message: Add articulated quadrotor camera mount

File: UAV_models/skydio_2/quadrotor.urdf (robot description, URDF)
Before this commit: robot quadrotor, 1 links, 0 joints
Links:
- added link camera_link, mass 0.005; visual box size=0.03 0.02 0.06; visual cylinder length=0.08 radius=0.0025
- added link camera_pitch_link, mass 0.005
Joints:
- added joint camera_optical_joint: type fixed, parent camera_pitch_link, child camera_link, origin xyz=0 0 0 rpy=-1.57079632679 0 -1.57079632679
- added joint camera_pitch_joint: type revolute, parent base_link, child camera_pitch_link, origin xyz=0.18 0 -0.03 rpy=0 0 0, axis 0 -1 0, limit lower=0.0 upper=1.57079632679 effort=1.0 velocity=4.0

Commit message: feat: integrate web GUI, stabilize flight controller, and add Dryden wind turbulence stub
- Unified Flask web GUI (joysticks, sliders, video stream)
- Fixed SE(3) controller mixer saturation bug that caused fly-aways
- Tuned PID gains properly using inertia matrix for stable hover and responsive yaw
- Implemented LCM bindings and communication for Web GUI
- Fixed video streaming buffer lag using background threads
- Removed duplicate properties in config YAML

File: UAV_models/skydio_2/quadrotor.urdf (robot description, URDF)
Before this commit: robot quadrotor, 3 links, 2 joints
Links:
- link base_link: mass 0.775 -> 0.765
- link camera_link: geometry 
